File: sch/airsens_p03/airsens_p03.kicad_sch (KiCad schematic)
At the start: 53 parts, among them J03 ADC_IN, Q1 BS170, U1 ME6211C33, U2 ESP32-WROOM-32

Commit message: central v0.1.18'
Parts:
- removed J?: MES_ON, symbol Connector:Conn_01x01_Male
- removed J?: MES_ON, symbol Connector:Conn_01x01_Female
- removed Q1: BS170, Package_TO_SOT_THT:TO-92_Inline, symbol Transistor_FET:BS170
- removed R7: 10k, symbol Device:R
- J?: value green_led -> yellow_led
- R4, R5, R6: value 1k -> 3.3k
- gave numbers to parts that had none: 3
- renumbered BME680 to j2
Other:
- moved on the sheet: D1, D2, D3, R4, R5, R6
