File: sch/airsens_p03/airsens_p03c.kicad_sch (KiCad schematic)
At the start: 47 parts, among them J03 ADC_IN, J1 ALIM, J3 USB TO UART, J4 PPK: power profiler kit, U1 ME6211C33, U2 ESP32-WROOM-32, j2 BME280

Commit message: proto p03c
Parts:
- removed D1: red, symbol Device:LED
- removed D2: green, symbol Device:LED
- removed D3: blue, symbol Device:LED
- removed J4: PPK: power profiler kit, symbol Connector_Generic:Conn_01x08
- removed J?: green_led, symbol Connector:Conn_01x01_Male
- removed J?: PPK_3, symbol Connector:Conn_01x01_Male
- removed J? (x2): red_led, symbol Connector:Conn_01x01_Male
- removed J?: PPK_0, symbol Connector:Conn_01x01_Male
- removed J? (x2): blue_led, symbol Connector:Conn_01x01_Male
- removed J?: PPK_4, symbol Connector:Conn_01x01_Male
- removed J?: yellow_led, symbol Connector:Conn_01x01_Male
- removed J?: PPK_2, symbol Connector:Conn_01x01_Male
- removed J?: PPK_1, symbol Connector:Conn_01x01_Male
- removed J?: PPK_5, symbol Connector:Conn_01x01_Male
- removed R4, R5, R6: 3.3k, symbol Device:R
Other:
- title: airsens proto 03 -> airsens proto 03b
- moved on the sheet: 4.5V, C1, C2, C3, C4, C5, EN, J1, J3, R1, R2, R3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

Commit message: proto P03abc
Other:
- title: airsens proto 03b -> airsens proto 03c-v1
Changed lines of the file:
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@@
   (paper "A4")
   (title_block
-    (title "airsens proto 03b")
-    (date "2022-07-10")
+    (title "airsens proto 03c-v1")
+    (date "2022-07-17")
     (rev "04")
     (company "JOM52")
